Commit message: [FEAT] Added RGBD camera
Added RGB camera to xacro and gazebo sensor with correct frame_id=chassis

File: urdf/my_robot.xacro (robot description, xacro)
@@ -148,4 +148,11 @@
     </collision>
   </link>
+  <joint name="camera_optical_joint" type="fixed">
+    <origin xyz="0 0 0" rpy="-1.5707 0 -1.5707"/>
+    <parent link="camera"/>
+    <child link="camera_link_optical"/>
+  </joint>
+  <link name="camera_link_optical">
+  </link>
   <joint type="fixed" name="hokuyo_joint">
     <origin xyz="0.15 0 0.07" rpy="0 0 0"/>
